Commit message: Rebase from 'debian/humble/andino_description'

File: urdf/andino.urdf.xacro (robot description, xacro)
@@ -21,4 +21,6 @@
   <xacro:property name="sensor_yaml" value="$(arg yaml_config_dir)/sensors.yaml" />
   <xacro:property name="sensor_prop" value="${xacro.load_yaml(sensor_yaml)}"/>
+  <xacro:property name="hardware_yaml" value="$(arg yaml_config_dir)/hardware.yaml" />
+  <xacro:property name="hardware_props" value="${xacro.load_yaml(hardware_yaml)}"/>
   <!-- Footprint link -->
   <xacro:footprint wheel_props="${wheel_props}" />
@@ -69,4 +71,5 @@
   <xacro:if value="$(arg use_real_ros_control)">
     <xacro:include filename="$(find ${package_name})/urdf/include/andino_control.urdf.xacro" />
+    <xacro:control hardware_props="${hardware_props}" />
   </xacro:if>
 </robot>

File: urdf/include/andino_control.urdf.xacro (robot description, xacro)
@@ -1,32 +1,37 @@
 <?xml version="1.0"?>
 <robot xmlns:xacro="http://www.ros.org/wiki/xacro">
-  <!-- TODO(francocipollone): This xacro should be part of andino_control package instead.-->
-  <ros2_control name="RealRobot" type="system">
-    <hardware>
-      <plugin>andino_base/DiffDriveAndino</plugin>
-      <!-- TODO(francocipollone): Parameters like loop_rate, device, baud_rate, etc should be loaded from a file or passed via the launch file as xacro args -->
-      <param name="left_wheel_name">left_wheel_joint</param>
-      <param name="right_wheel_name">right_wheel_joint</param>
-      <param name="serial_device">/dev/ttyUSB_ARDUINO</param>
-      <param name="baud_rate">57600</param>
-      <param name="timeout">1000</param>
-      <param name="enc_ticks_per_rev">585</param>
-    </hardware>
-    <joint name="left_wheel_joint">
-      <command_interface name="velocity">
-        <param name="min">-5</param>
-        <param name="max">5</param>
-      </command_interface>
-      <state_interface name="velocity"/>
-      <state_interface name="position"/>
-    </joint>
-    <joint name="right_wheel_joint">
-      <command_interface name="velocity">
-        <param name="min">-5</param>
-        <param name="max">5</param>
-      </command_interface>
-      <state_interface name="velocity"/>
-      <state_interface name="position"/>
-    </joint>
-  </ros2_control>
+<!-- ===================== Control xacro =========================================
+  params:
+  - hardware_props [dictionary]: hardware properties loaded from the YAML file.
+-->
+  <xacro:macro name="control" params="hardware_props" >
+    <!-- TODO(francocipollone): This xacro should be part of andino_control package instead.-->
+    <ros2_control name="RealRobot" type="system">
+      <hardware>
+        <plugin>andino_base/DiffDriveAndino</plugin>
+        <param name="left_wheel_name">${hardware_props['left_wheel_name']}</param>
+        <param name="right_wheel_name">${hardware_props['right_wheel_name']}</param>
+        <param name="serial_device">${hardware_props['serial_device']}</param>
+        <param name="baud_rate">${hardware_props['baud_rate']}</param>
+        <param name="timeout">${hardware_props['timeout']}</param>
+        <param name="enc_ticks_per_rev">${hardware_props['enc_ticks_per_rev']}</param>
+      </hardware>
+      <joint name="left_wheel_joint">
+        <command_interface name="velocity">
+          <param name="min">-5</param>
+          <param name="max">5</param>
+        </command_interface>
+        <state_interface name="velocity"/>
+        <state_interface name="position"/>
+      </joint>
+      <joint name="right_wheel_joint">
+        <command_interface name="velocity">
+          <param name="min">-5</param>
+          <param name="max">5</param>
+        </command_interface>
+        <state_interface name="velocity"/>
+        <state_interface name="position"/>
+      </joint>
+    </ros2_control>
+  </xacro:macro>
 </robot>
